File: pico-zero-base.kicad/pico-zero-base.kicad_pcb (KiCad board)
At the start: 2 copper layers, 65 x 30 mm, 7 parts, among them J1 GPIO, SW1 SW_Push_SLIM, U1 Pico

Commit message: add optional pullups Rev 1.2
Parts:
- added R1: 10K, Resistor_SMD:R_1206_3216Metric_Pad1.30x1.75mm_HandSolder, B.Cu at (115.3, 85.1)
- added R2: 10K, Resistor_SMD:R_1206_3216Metric_Pad1.30x1.75mm_HandSolder, B.Cu at (118.9, 87.6)
Routing:
- net +3.3V: track 28.0 -> 43.5 mm, vias 0 -> 1
- net /GPIO[3]/SCL1: track 24.4 -> 25.9 mm
- net /GPIO[2]/SDA1: track 24.4 -> 25.8 mm
Other:
- board text added: "Rev 1.2"
- board text removed: "Rev 1.1"

Commit message: pico-zero-base: Rev 2.0
Connections:
- U1 pad 21: /GPIO[19]/PCM.FS -> /GPIO[21]/PCM.DOUT
- U1 pad 22: /GPIO[16] -> /GPIO[20]/PCM.DIN
- U1 pad 24: /GPIO[21]/PCM.DOUT -> /GPIO[18]/PCM.CLK
- U1 pad 25: /GPIO[20]/PCM.DIN -> /GPIO[19]/PCM.FS
- U1 pad 26: /GPIO[12]/PWM0 -> /GPIO[16]
- U1 pad 27: /GPIO[5] -> /GPIO[12]/PWM0
- U1 pad 29: /GPIO[7]/SPI0.CE1 -> /GPIO[5]
- U1 pad 31: /GPIO[25] -> /GPIO[7]/SPI0.CE1
- U1 pad 32: /GPIO[24] -> /GPIO[25]
- U1 pad 34: /GPIO[18]/PCM.CLK -> /GPIO[24]
Routing:
- net /GPIO[18]/PCM.CLK: track 8.15 -> 35.5 mm
- net /GPIO[21]/PCM.DOUT: track 17.6 -> 8.01 mm
- net /GPIO[7]/SPI0.CE1: track 8.11 -> 15.2 mm
- net /GPIO[20]/PCM.DIN: track 14.4 -> 8.06 mm
- net /GPIO[24]: track 8.01 -> 14.1 mm
- net /GPIO26: track 29.9 -> 35.0 mm
- net /GPIO[5]: track 5.57 -> 9.72 mm
- net /GPIO[16]: track 8.15 -> 11.8 mm
- net /GPIO[12]/PWM0: track 8.11 -> 10.1 mm
- net /RESET: track 48.2 -> 47.4 mm
- net /GPIO[6]: track 37.8 -> 37.1 mm
- net /GPIO[19]/PCM.FS: track 8.62 -> 8.42 mm, vias 1 -> 0
Other:
- board text added: "Rev 2.0"
- board text removed: "Rev 1.2"
