File: pico-zero-base.kicad/pico-zero-base.kicad_sch (KiCad schematic)
At the start: 5 parts, among them J1 GPIO, SW1 SW_Push_SLIM, U1 Pico

Commit message: pico-zero-base: Rev 2.0
Connections:
- net GPIO[12]/PWM0: now also U1.27 (GPIO21); no longer U1.26 (GPIO20)
- net GPIO[16]: now also U1.26 (GPIO20); no longer U1.22 (GPIO17)
- net GPIO[18]/PCM.CLK: now also U1.24 (GPIO18); no longer U1.34 (GPIO28_ADC2)
- net GPIO[19]/PCM.FS: now also U1.25 (GPIO19); no longer U1.21 (GPIO16)
- net GPIO[20]/PCM.DIN: now also U1.22 (GPIO17); no longer U1.25 (GPIO19)
- net GPIO[21]/PCM.DOUT: now also U1.21 (GPIO16); no longer U1.24 (GPIO18)
- net GPIO[24]: now also U1.34 (GPIO28_ADC2); no longer U1.32 (GPIO27_ADC1)
- net GPIO[25]: now also U1.32 (GPIO27_ADC1); no longer U1.31 (GPIO26_ADC0)
- net GPIO[5]: now also U1.29 (GPIO22); no longer U1.27 (GPIO21)
- net GPIO[7]/SPI0.CE1: now also U1.31 (GPIO26_ADC0); no longer U1.29 (GPIO22)
Changed lines of the file:
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@@
   (title_block
     (title "pico-zero-base")
-    (date "2023-04-07")
-    (rev "1.2")
+    (date "2023-04-29")
+    (rev "2.0")
     (company "Bernhard Bablok")
     (comment 1 "https://github.com/bablokb/pcb-pi-pico-base")
@@
     (effects (font (size 1.27 1.27)) (justify right bottom))
   )
-  (label "GPIO[25]" (at 100.33 128.905 0)
+  (label "GPIO[25]" (at 100.33 126.365 0)
     (effects (font (size 1.27 1.27)) (justify left bottom))
   )
@@
     (effects (font (size 1.27 1.27)) (justify left bottom))
   )
-  (label "GPIO[24]" (at 100.33 126.365 0)
+  (label "GPIO[24]" (at 100.33 121.285 0)
     (effects (font (size 1.27 1.27)) (justify left bottom))
   )
@@
     (effects (font (size 1.27 1.27)) (justify right bottom))
   )
-  (label "GPIO[21]{slash}PCM.DOUT" (at 100.33 146.685 0)
+  (label "GPIO[21]{slash}PCM.DOUT" (at 100.33 154.305 0)
     (effects (font (size 1.27 1.27)) (justify left bottom))
   )
@@
     (effects (font (size 1.27 1.27)) (justify right bottom))
   )
-  (label "GPIO[12]{slash}PWM0" (at 100.33 141.605 0)
+  (label "GPIO[12]{slash}PWM0" (at 100.33 139.065 0)
     (effects (font (size 1.27 1.27)) (justify left bottom))
   )
@@
     (effects (font (size 1.27 1.27)) (justify left bottom))
   )
-  (label "GPIO[16]" (at 100.33 151.765 0)
+  (label "GPIO[16]" (at 100.33 141.605 0)
     (effects (font (size 1.27 1.27)) (justify left bottom))
   )
@@
     (effects (font (size 1.27 1.27)) (justify left bottom))
   )
-  (label "GPIO[19]{slash}PCM.FS" (at 100.33 154.305 0)
+  (label "GPIO[19]{slash}PCM.FS" (at 100.33 144.145 0)
     (effects (font (size 1.27 1.27)) (justify left bottom))
   )
@@
     (effects (font (size 1.27 1.27)) (justify right bottom))
   )
-  (label "GPIO[20]{slash}PCM.DIN" (at 100.33 144.145 0)
+  (label "GPIO[20]{slash}PCM.DIN" (at 100.33 151.765 0)
     (effects (font (size 1.27 1.27)) (justify left bottom))
   )
@@
     (effects (font (size 1.27 1.27)) (justify right bottom))
   )
-  (label "GPIO[7]{slash}SPI0.CE1" (at 100.33 133.985 0)
+  (label "GPIO[7]{slash}SPI0.CE1" (at 100.33 128.905 0)
     (effects (font (size 1.27 1.27)) (justify left bottom))
   )
@@
     (effects (font (size 1.27 1.27)) (justify right bottom))
   )
-  (label "GPIO[5]" (at 100.33 139.065 0)
+  (label "GPIO[5]" (at 100.33 133.985 0)
     (effects (font (size 1.27 1.27)) (justify left bottom))
   )
@@
     (effects (font (size 1.27 1.27)) (justify left bottom))
   )
-  (label "GPIO[18]{slash}PCM.CLK" (at 100.33 121.285 0)
-    (effects (font (size 1.27 1.27)) (justify left bottom))
-  )
+  (label "GPIO[18]{slash}PCM.CLK" (at 100.33 146.685 0)
+    (effects (font (size 1.27 1.27)) (justify left bottom))
+  )
